File: hs-32-spi-3d.brd (EAGLE design)
At the start: 15.2 x 23.5 mm, 24 parts, among them U1 RHD2132_QFN, U2 BNO055, U3 TLV70725

Commit message: Increased minimum drill to 0.25 mm.
Also created a pad for the AUXIN3.
Parts:
- added AUX3: TESTPOINT_SMALL, RHD2000_eval_board:TESTPOINT_SMALL
Connections:
- removed net XOUT: U1.14
- removed net YOUT: U1.15
- removed net ZOUT: U1.16
- new net AUXIN3: AUX3.1, U1.16
- net VCC: now also U1.14, U1.15
Routing:
- net AUXIN3: track 0.00 -> 5.32 mm, vias 0 -> 1
- net VCC: track 13.5 -> 15.5 mm
- net GND: vias 27 -> 32

Commit message: Corrected C6 and C7 values to 4.7uF.
Parts:
- C6: value 1u -> 4.7u
- C7: value 1uF -> 4.7uF
Changed lines of the file:
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@@
 <attribute name="NAME" x="14.9479" y="17.4752" size="0.8128" layer="25" font="vector" ratio="18" rot="R90"/>
 </element>
-<element name="C6" library="jonnew" package="0402" value="1u" x="13.081" y="6.2865" smashed="yes">
+<element name="C6" library="jonnew" package="0402" value="4.7u" x="13.081" y="6.2865" smashed="yes">
 <attribute name="NAME" x="15.0495" y="5.4102" size="0.8128" layer="25" font="vector" ratio="18" rot="R90"/>
 <attribute name="VALUE" x="11.811" y="4.5085" size="1.016" layer="27" font="vector" ratio="18"/>
@@
 <attribute name="NAME" x="3.745" y="0.7362" size="0.6096" layer="25" font="vector" ratio="18"/>
 </element>
-<element name="C7" library="jonnew" package="0402T" value="1uF" x="5.6134" y="1.2192" smashed="yes" rot="R90">
+<element name="C7" library="jonnew" package="0402T" value="4.7uF" x="5.6134" y="1.2192" smashed="yes" rot="R90">
 <attribute name="NAME" x="5.9952" y="0.3572" size="0.8128" layer="25" font="vector" ratio="18"/>
 <attribute name="PARTNO" value="CL05A105KO5NNNC" x="14.5034" y="-3.5433" size="1.778" layer="27" rot="R90" display="off"/>
