File: hs-32-spi-3d.sch (EAGLE design)
At the start: 25 parts, among them U1 RHD2132_QFN, U2 BNO055, U3 TLV70725

Commit message: Added EEPROM.
Parts:
- added U4: 24CW640T-I/CS0668, 24CW640T-I_CS0668:24CW640T-I/CS0668
Connections:
- net +2V5: now also U4.VCC
- net BNO_SCL: now also U4.SCL
- net BNO_SDA: now also U4.SDA
- net GND: now also U4.GND
Changed lines of the file:
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@@
 <layer number="59" name="tCarbon" color="7" fill="1" visible="no" active="no"/>
 <layer number="60" name="bCarbon" color="7" fill="1" visible="no" active="no"/>
+<layer number="88" name="SimResults" color="9" fill="1" visible="yes" active="yes"/>
+<layer number="89" name="SimProbes" color="9" fill="1" visible="yes" active="yes"/>
 <layer number="90" name="Modules" color="5" fill="1" visible="yes" active="yes"/>
 <layer number="91" name="Nets" color="2" fill="1" visible="yes" active="yes"/>
@@
 <part name="P+11" library="supply1" deviceset="VCC" device=""/>
 <part name="AUX3" library="RHD2000_eval_board" deviceset="TESTPOINT" device="_SMALL"/>
+<part name="U4" library="24CW640T-I_CS0668" deviceset="24CW640T-I/CS0668" device=""/>
+<part name="GND16" library="supply1" deviceset="GND" device=""/>
+<part name="U$7" library="jonnew" deviceset="+2V5" device=""/>
 </parts>
 <sheets>
@@
 <attribute name="NAME" x="40.894" y="126.365" size="1.778" layer="95"/>
 </instance>
+<instance part="U4" gate="G$1" x="337.82" y="175.26" smashed="yes"/>
+<instance part="GND16" gate="1" x="353.06" y="154.94" smashed="yes">
+<attribute name="VALUE" x="350.52" y="152.4" size="1.778" layer="96"/>
+</instance>
+<instance part="U$7" gate="G$1" x="353.06" y="193.04" smashed="yes"/>
 </instances>
 <busses>
@@
 <pinref part="GND15" gate="1" pin="GND"/>
 </segment>
+<segment>
+<pinref part="U4" gate="G$1" pin="GND"/>
+<wire x1="347.98" y1="170.18" x2="353.06" y2="170.18" width="0.1524" layer="91"/>
+<pinref part="GND16" gate="1" pin="GND"/>
+<wire x1="353.06" y1="170.18" x2="353.06" y2="157.48" width="0.1524" layer="91"/>
+</segment>
 </net>
 <net name="VCC" class="0">
@@
 <label x="284.48" y="99.06" size="1.27" layer="95" rot="R180" xref="yes"/>
 <pinref part="U2" gate="G$1" pin="COM1/SCL/RX"/>
+<label x="325.12" y="180.34" size="1.27" layer="95" rot="R180" xref="yes"/>
 </segment>
 <segment>
@@
 <wire x1="109.22" y1="60.96" x2="109.22" y2="43.18" width="0.1524" layer="91"/>
 </segment>
+<segment>
+<pinref part="U4" gate="G$1" pin="SCL"/>
+<wire x1="327.66" y1="180.34" x2="325.12" y2="180.34" width="0.1524" layer="91"/>
+</segment>
 </net>
 <net name="BNO_SDA" class="0">
@@
 <label x="284.48" y="96.52" size="1.27" layer="95" rot="R180" xref="yes"/>
 <pinref part="U2" gate="G$1" pin="COM0/SDA/TX"/>
+<label x="325.12" y="172.72" size="1.27" layer="95" rot="R180" xref="yes"/>
 </segment>
 <segment>
@@
 <wire x1="127" y1="63.5" x2="106.68" y2="63.5" width="0.1524" layer="91"/>
 <wire x1="106.68" y1="63.5" x2="106.68" y2="43.18" width="0.1524" layer="91"/>
+</segment>
+<segment>
+<pinref part="U4" gate="G$1" pin="SDA"/>
+<wire x1="327.66" y1="172.72" x2="325.12" y2="172.72" width="0.1524" layer="91"/>
 </segment>
 </net>
@@
 <wire x1="149.86" y1="93.98" x2="149.86" y2="91.44" width="0.1524" layer="91"/>
 </segment>
-</net>
+<segment>
+<pinref part="U4" gate="G$1" pin="VCC"/>
+<wire x1="347.98" y1="180.34" x2="353.06" y2="180.34" width="0.1524" layer="91"/>
+<pinref part="U$7" gate="G$1" pin="+2V5"/>
+<wire x1="353.06" y1="180.34" x2="353.06" y2="193.04" width="0.1524" layer="91"/>
+</segment>
+</net>

Commit message: Minor details regarding capacitors' nomenclature.
Parts:
- C3, C4, C5: value 0.1uF -> 100nF
- C6: value 4.7u -> 4.7uF
Changed lines of the file:
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@@
 <part name="GND10" library="supply1" deviceset="GND" device=""/>
 <part name="REF" library="RHD2000_eval_board" deviceset="TESTPOINT" device="_SMALL"/>
-<part name="C6" library="jonnew" deviceset="C" device="_0402" value="4.7u"/>
-<part name="C4" library="jonnew" deviceset="C" device="_0402T" value="0.1uF"/>
-<part name="C3" library="jonnew" deviceset="C" device="_0402T" value="0.1uF"/>
-<part name="C5" library="jonnew" deviceset="C" device="_0201T" value="0.1uF"/>
+<part name="C6" library="jonnew" deviceset="C" device="_0402" value="4.7uF"/>
+<part name="C4" library="jonnew" deviceset="C" device="_0402T" value="100nF"/>
+<part name="C3" library="jonnew" deviceset="C" device="_0402T" value="100nF"/>
+<part name="C5" library="jonnew" deviceset="C" device="_0201T" value="100nF"/>
 <part name="U3" library="jonnew" deviceset="TLV707" device="" value="TLV70725"/>
 <part name="U$45" library="jonnew" deviceset="+2V5" device=""/>
